File: KiCad/TallyLight/TallyLight.kicad_sch (KiCad schematic)
At the start: 4 parts, among them IC1 ATMEGA328PB-AU, IC2 VEML7700-TT, J1 USB4125-GF-A-0190

Commit message: Minor Updates to schematic
Parts:
- added C1, C3: CL21B105KBFNNNG, SamacSys_Parts:CAPC2012X135N, symbol SamacSys_Parts:CL21B105KBFNNNG
- added C10, C4, C5, C6, C7, C8, C9: C0805C104M5RACTU, SamacSys_Parts:C0805, symbol SamacSys_Parts:C0805C104M5RACTU
- added C2: C0805C471K5RACTU, SamacSys_Parts:C0805, symbol SamacSys_Parts:C0805C471K5RACTU
- added IC3: TC1263-3.3VOATR, SamacSys_Parts:SOIC127P600X175-8N, symbol SamacSys_Parts:TC1263-3.3VOATR
- added Q1: BSS138DW-7-F, SOT65P210X110-6N, symbol SamacSys_Parts:BSS138DW-7-F
- added RN1: YC124-JR-0710KL, YC124JR0710KL, symbol SamacSys_Parts:YC124-JR-0710KL
- added U1, U2, U3, U4, U5, U6, U7, U8: ~, symbol Samuel_Library:SK6812_SIDE-A
- added U9: NRF24L01, symbol MySensors:NRF24L01
Connections:
- net GND: now reaches J1.A12 (GND_1)
- net GND: now also IC1.21 (GND_2), IC1.5 (GND_1), IC2.3 (GND), J1.B12 (GND_2), S1.C1, S1.C2, C1.2, C10.1, C2.2, C3.2, C4.1, C5.1, C6.1, C7.1, C8.1, C9.1, IC3.2 (GND), U1.4 (GND), U2.4 (GND), U3.4 (GND), U5.4 (GND), U6.4 (GND), U7.4 (GND), U8.4 (GND), U9.1 (GND)
- net +5V: now reaches J1.A9 (VBUS_1)
- net +5V: now also IC1.4 (VCC), J1.B9 (VBUS_2), C10.2, C3.1, C4.2, C5.2, C6.2, C7.2, C8.2, C9.2, IC3.6 (~{SHDN}), IC3.8 (VIN), RN1.7, RN1.8, U1.2 (VDD), U2.2 (VDD), U3.2 (VDD), U4.2 (VDD), U5.2 (VDD), U6.2 (VDD), U7.2 (VDD), U8.2 (VDD)
- net HEX_1: now reaches S1.1
- net HEX_1: now also IC1.23 (PC0_(ADC0/PTCY/MISO1))
- net HEX_2: now reaches S1.2
- net HEX_2: now also IC1.24 (PC1_(ADC1/PTCY/SCK1))
- net HEX_4: now reaches S1.4
- net HEX_4: now also IC1.25 (PC2_(ADC2/PTCY))
- net HEX_8: now reaches S1.8
- net HEX_8: now also IC1.26 (PC3_(ADC3/PTCY))
- net SCL_3V: now reaches IC2.1 (SCL)
- net SCL_3V: now also Q1.1 (S2), RN1.3
- net +3V3: now reaches IC2.2 (VDD)
- net +3V3: now also C1.1, IC3.1 (VOUT), Q1.2 (G2), Q1.5 (G1), RN1.5, RN1.6, U9.2 (VCC)
- net SDA_3V: now reaches IC2.4 (SDA)
- net SDA_3V: now also Q1.4 (S1), RN1.4
- net LED_DATA: now reaches IC1.12 ((ICP1/CLKO/PTCXY)_PB0)
- net LED_DATA: now also U1.1 (DIN)
- net RF_CE: now reaches IC1.13 ((OC1A/PTCXY)_PB1)
- net RF_CE: now also U9.3 (CE)
- net RF_CSN: now reaches IC1.14 ((~{SS0}/OC1B/PTCXY)_PB2)
- net RF_CSN: now also U9.4 (CSN)
- net MOSI: now reaches IC1.15 ((MOSI0/TXD1/OC2A/PTCXY)_PB3)
- net MOSI: now also U9.6 (MOSI)
- net MISO: now reaches IC1.16 ((MISO0/RXD1/PTCXY)_PB4)
- net MISO: now also U9.7 (MISO)
- net SCK: now reaches IC1.17 (PB5_(PTCXY/XCK0/SCK0))
- net SCK: now also U9.5 (SCK)
- net SDA: now reaches IC1.27 (PC4_(ADC4/PTCY/SDA0))
- net SDA: now also Q1.3 (D1), RN1.2
- net SCL: now reaches IC1.28 (PC5_(ADC5/PTCY/SCL0))
- net SCL: now also Q1.6 (D2), RN1.1
- new net: U1.3 (DOUT), U2.1 (DIN)
- new net: U2.3 (DOUT), U3.1 (DIN)
- new net: U7.3 (DOUT), U8.1 (DIN)
- new net: U4.3 (DOUT), U5.1 (DIN)
- new net: U5.3 (DOUT), U6.1 (DIN)
- new net: U3.3 (DOUT), U4.1 (DIN)
- new net: C2.1, IC3.4 (BYPASS)
- new net: U6.3 (DOUT), U7.1 (DIN)
- no-connect marks 0 -> 9
Other:
- note added: "HEX SWITCH"
- note added: "LUX SENSOR"
- note added: "PIXEL LEDS"
- note added: "POWER"
- note added: "RADIO"
- moved on the sheet: IC2, J1, S1

Commit message: Made a PCB, added error status on LEDs at power up, probably did many more code changes since the last commit
Parts:
- added 3V1, 5V1, LED1: LED, LED_SMD:LED_0805_2012Metric, symbol Device:LED
- added C12, C13: 106, SamacSys_Parts:CAPC1608X90N, symbol SamacSys_Parts:GRM188D71A106MA73J
- added C14, C15, C16, C8: 104, SamacSys_Parts:C0805, symbol SamacSys_Parts:C0805C104M5RACTU
- added C17, C18: 22p, SamacSys_Parts:C0805, symbol SamacSys_Parts:C0805C220K5HACTU
- added J2: Conn_01x01_Pin, Connector_PinSocket_2.54mm:PinSocket_1x01_P2.54mm_Vertical, symbol Connector:Conn_01x01_Pin
- added J3: Conn_01x06_Pin, Connector_PinHeader_2.54mm:PinHeader_1x06_P2.54mm_Vertical, symbol Connector:Conn_01x06_Pin
- added J4: Conn_01x03_Pin, Connector_PinHeader_2.54mm:PinHeader_1x03_P2.54mm_Vertical, symbol Connector:Conn_01x03_Pin
- added R1, R2: 5K1, Samuel_Library:R_0805_2012Metric_Pad1.20x1.40mm_HandSolder, symbol Device:R
- added R3: 100K, Samuel_Library:R_0805_2012Metric_Pad1.20x1.40mm_HandSolder, symbol Device:R
- added R4: 130R, Samuel_Library:R_0805_2012Metric_Pad1.20x1.40mm_HandSolder, symbol Device:R
- added R5, R6: 300R, Samuel_Library:R_0805_2012Metric_Pad1.20x1.40mm_HandSolder, symbol Device:R
- added SET1: TS02-66-50-BK-260-SCR-D, SamacSys_Parts:TS026650BK260SCRD, symbol SamacSys_Parts:TS02-66-50-BK-260-SCR-D
- added Y1: 16M, SamacSys_Parts:ABLS, symbol SamacSys_Parts:ABLS-16.000MHz-16-A-4-H-T
- C1: renamed from C4; value C0805C104M5RACTU -> 104
- C10: renamed from C2; value C0805C471K5RACTU -> 471
- C11: renamed from C3; value CL21B105KBFNNNG -> 105
- C2: renamed from C5; value C0805C104M5RACTU -> 104
- C3: renamed from C6; value C0805C104M5RACTU -> 104
- C4: renamed from C7; value C0805C104M5RACTU -> 104
- C5: renamed from C8; value C0805C104M5RACTU -> 104
- C6: renamed from C9; value C0805C104M5RACTU -> 104
- C7: renamed from C10; value C0805C104M5RACTU -> 104
- C9: renamed from C1; value CL21B105KBFNNNG -> 105
- IC2: footprint VEML7700 -> SamacSys_Parts:VEML7700
- IC3: renamed from IC1; footprint QFP80P900X900X120-32N -> SamacSys_Parts:QFP80P900X900X120-32N
- J1: footprint USB4125GFA0190 -> SamacSys_Parts:USB4125GFA0190
- Q1: footprint SOT65P210X110-6N -> SamacSys_Parts:SOT65P210X110-6N
- RN1: value YC124-JR-0710KL -> 10K; footprint YC124JR0710KL -> SamacSys_Parts:YC124JR0710KL
- TALLY#1: renamed from S1; footprint SD1210 -> SamacSys_Parts:SD1210
- U1: value ~ -> LED 1; footprint (none) -> Samuel_Library:SK6812_SIDE-A
- U2: value ~ -> LED 2; footprint (none) -> Samuel_Library:SK6812_SIDE-A
- U3: value ~ -> LED 3; footprint (none) -> Samuel_Library:SK6812_SIDE-A
- U4: value ~ -> LED 4; footprint (none) -> Samuel_Library:SK6812_SIDE-A
- U5: value ~ -> LED 5; footprint (none) -> Samuel_Library:SK6812_SIDE-A
- U6: value ~ -> LED 6; footprint (none) -> Samuel_Library:SK6812_SIDE-A
- U7: value ~ -> LED 7; footprint (none) -> Samuel_Library:SK6812_SIDE-A
- U8: value ~ -> LED 8; footprint (none) -> Samuel_Library:SK6812_SIDE-A
- U9: footprint (none) -> MySensors:NRF24L01-SMD
- renumbered IC3 to IC1
Connections:
- net +3V3: now also 3V1.1 (K), C12.1
- net +5V: now also IC3.18 (AVCC), 5V1.1 (K), C13.1, C14.2, C8.2, J3.4 (Pin_4), J4.1 (Pin_1), R3.1
- net GND: now also U4.4 (GND), C12.2, C13.2, C14.1, C16.2, C17.1, C18.1, C8.1, J3.5 (Pin_5), J3.6 (Pin_6), J4.3 (Pin_3), R1.2, R2.2, R4.1, R5.1, R6.1, SET1.3 (COM_1), SET1.4 (COM_2)
- net at J1.A5 (CC1): now also R1.1
- net at J1.B5 (CC2): now also R2.1
- net BTN: now reaches IC3.10 ((OC0A/PTCXY/AIN0)_PD6)
- net BTN: now also SET1.2 (NO_2)
- net LED_DATA_2: now reaches IC3.11 ((PTCXY/AIN1)_PD7)
- net LED_DATA_2: now also J4.2 (Pin_2)
- net at IC3.20 (AREF): now also C16.1
- net RST: now reaches IC3.29 (PC6_(~{RESET}))
- net RST: now also C15.1, R3.2
- net RXI: now reaches IC3.30 (PD0_(PTCXY/OC3A/RXD0))
- net RXI: now also J3.3 (Pin_3)
- net TXO: now reaches IC3.31 (PD1_(PTCXY/OC4A/TXD0))
- net TXO: now also J3.2 (Pin_2)
- net at IC3.32 (PD2_(PTCXY/INT0/OC3B/OC4B)): now also J2.1 (Pin_1)
- net XTAL1: now reaches IC3.7 ((XTAL1/TOSC1)_PB6)
- net XTAL1: now also C17.2, Y1.1
- net XTAL2: now reaches IC3.8 ((XTAL2/TOSC2)_PB7)
- net XTAL2: now also C18.2, Y1.2
- net LED: now reaches IC3.9 ((OC0B/T1/PTCXY)_PD5)
- net LED: now also LED1.2 (A)
- new net: 5V1.2 (A), R5.2
- new net: LED1.1 (K), R6.2
- new net: 3V1.2 (A), R4.2
- new net DTR: C15.2, J3.1 (Pin_1)
- no-connect marks 9 -> 16
